Commit message: add imu

File: urdf/alphasense.urdf.xacro (robot description, xacro)
@@ -20,4 +20,19 @@
     </inertial>
   </link>
+  <link name="imu_link">
+    <visual>
+      <geometry>
+        <box size="3e-3 2e-3 1e-3" />
+      </geometry>
+      <material name="black">
+        <color rgba="0 0 0 1" />
+      </material>
+    </visual>
+  </link>
+  <joint name="imu_joint" type="fixed">
+    <origin xyz="6e-3 -8.55e-3 17.4e-3" rpy="${pi} 0 0"/>
+    <parent link="alphasense_mount" />
+    <child link="imu_link" />
+  </joint>
   </xacro:macro>
 </robot>

Commit message: add all cameras into urdf

File: urdf/alphasense.urdf.xacro (robot description, xacro)
@@ -35,4 +35,69 @@
     <child link="imu_link" />
   </joint>
+  <link name="cam_front_left">
+    <visual>
+      <geometry>
+        <box size="1e-3 1e-3 1e-3" />
+      </geometry>
+      <material name="black">
+        <color rgba="0 0 0 1" />
+      </material>
+    </visual>
+  </link>
+  <link name="cam_front_right">
+    <visual>
+      <geometry>
+        <box size="1e-3 1e-3 1e-3" />
+      </geometry>
+      <material name="black">
+        <color rgba="0 0 0 1" />
+      </material>
+    </visual>
+  </link>
+  <link name="cam_side_right">
+    <visual>
+      <geometry>
+        <box size="1e-3 1e-3 1e-3" />
+      </geometry>
+      <material name="black">
+        <color rgba="0 0 0 1" />
+      </material>
+    </visual>
+  </link>
+  <link name="cam_side_left">
+    <visual>
+      <geometry>
+        <box size="1e-3 1e-3 1e-3" />
+      </geometry>
+      <material name="black">
+        <color rgba="0 0 0 1" />
+      </material>
+    </visual>
+  </link>
+  <!-- front right camera which is cam0 in alphasense driver -->
+  <joint name="front_right_cam_joint" type="fixed">
+    <origin xyz="0.0438 0.0485 -0.0109" rpy="1.5708 0.0043 1.5675 "/>
+    <parent link="imu_link" />
+    <child link="cam_front_right" />
+  </joint>
+  <!-- front left camera which is cam1 in alphasense driver -->
+  <joint name="front_left_cam_joint" type="fixed">
+    <origin xyz="0.0437 -0.0611 -0.0115" rpy=" 1.5715 -0.0042 1.5712 "/>
+    <parent link="imu_link" />
+    <child link="cam_front_left" />
+  </joint>
+  <!-- top camera which is cam2 in alphasense driver, haven't calibrated yet -->
+  <!-- side right camera which is cam3 in alphasense driver -->
+  <joint name="side_right_cam_joint" type="fixed">
+    <origin xyz="-0.006 0.061 -0.0104" rpy="1.571 0.0 3.14"/>
+    <parent link="imu_link" />
+    <child link="cam_side_right" />
+  </joint>
+  <!-- side left camera which is cam4 in alphasense driver -->
+  <joint name="side_left_cam_joint" type="fixed">
+    <origin xyz="-0.00789 -0.07720 -0.01356" rpy="1.5733 0.00443 -0.0052"/>
+    <parent link="imu_link" />
+    <child link="cam_side_left" />
+  </joint>
   </xacro:macro>
 </robot>

Commit message: update side cam right with kalibr values

File: urdf/alphasense.urdf.xacro (robot description, xacro)
@@ -90,5 +90,5 @@
   <!-- side right camera which is cam3 in alphasense driver -->
   <joint name="side_right_cam_joint" type="fixed">
-    <origin xyz="-0.006 0.061 -0.0104" rpy="1.571 0.0 3.14"/>
+    <origin xyz="-0.006 0.062 -0.0105" rpy="1.5691 -0.0061 3.1334"/>
     <parent link="imu_link" />
     <child link="cam_side_right" />

Commit message: add os_imu link from Kalibr

File: urdf/alphasense.urdf.xacro (robot description, xacro)
@@ -75,4 +75,20 @@
     </visual>
   </link>
+  <link name="os_imu">
+    <visual>
+      <geometry>
+        <box size="1e-3 1e-3 1e-3" />
+      </geometry>
+      <material name="black">
+        <color rgba="0 0 0 1" />
+      </material>
+    </visual>
+  </link>
+  <!-- obtained from Kalibr which is different with the datasheet-->
+  <joint name="os_imu_joint" type="fixed">
+    <origin xyz="-0.05072 -0.02064 -0.04077" rpy="3.13503 -0.00927 -0.00483"/>
+    <parent link="imu_link" />
+    <child link="os_imu" />
+  </joint>
   <!-- front right camera which is cam0 in alphasense driver -->
   <joint name="front_right_cam_joint" type="fixed">
