Commit message: update camera transforms and readme

File: urdf/halo.urdf (robot description, URDF)
Before this commit: robot halo, 9 links, 8 joints
Joints:
- joint front_left_cam_joint: origin xyz=0.0437 -0.0611 -0.0115 rpy= 1.5715 -0.0042 1.5712  -> xyz=0.0457 -0.0642 -0.0102 rpy= 1.5698 -0.0023 1.5609 
- joint front_right_cam_joint: origin xyz=0.0438 0.0485 -0.0109 rpy=1.5708 0.0043 1.5675  -> xyz=0.0462 0.0469 -0.0094 rpy=1.5630 0.0066 1.5719
- joint imu_joint: origin xyz=6e-3 -8.55e-3 17.4e-3 rpy=3.141592653589793 0 0 -> xyz=6e-3 -8.55e-3 17.4e-3 rpy=${pi} 0 0
- joint side_left_cam_joint: origin xyz=-0.00789 -0.07720 -0.01356 rpy=1.5733 0.00443 -0.0052 -> xyz=-0.0072 -0.0754 -0.0113 rpy=1.5707 0.0045 -0.0076
- joint side_right_cam_joint: origin xyz=-0.006 0.062 -0.0105 rpy=1.5691 -0.0061 3.1334 -> xyz=-0.0058 0.0526 -0.0117 rpy=1.5603 -0.0067 3.1407

File: urdf/halo.urdf.xacro (robot description, xacro)
@@ -14,5 +14,5 @@
     </visual>
   </link>
-  <joint name="handle_to_base_mount" type="fixed">
+  <joint name="body_to_base_mount" type="fixed">
     <origin xyz="0 0 0" rpy="0 0 0" />
     <parent link="base" />

Commit message: load the alphasense from outside

File: urdf/halo.urdf (robot description, URDF)
Before this commit: robot halo, 9 links, 8 joints
Links:
- removed link handle
- added link body; visual mesh filename=package://halo_description/urdf/meshes/halo_body.dae
Joints:
- joint base_to_alphasense: origin xyz=0 0 0 rpy=0 0 0 -> xyz=32e-3 0.15e-3 47.7e-3 rpy=0 0 0
- joint base_to_ouster: origin xyz=-59e-3 0 51e-3 rpy=0 0 0 -> xyz=1e-3 0 90.683e-3 rpy=0 0 0
- joint handle_to_base_mount: child handle -> body

File: urdf/halo.urdf.xacro (robot description, xacro)
@@ -1,5 +1,5 @@
 <?xml version="1.0" ?>
 <robot name="halo" xmlns:xacro="http://www.ros.org/wiki/xacro">
-  <xacro:include filename="$(find halo_description)/urdf/alphasense.urdf.xacro" />
+  <xacro:include filename="$(find alphasense_description)/urdf/alphasense.urdf.xacro" />
   <xacro:include filename="$(find ouster_description)/urdf/ouster.urdf.xacro" />
   <link name="base" />
@@ -7,4 +7,21 @@
     <origin xyz="32e-3 0.15e-3 47.7e-3" rpy="0 0 0" />
   </xacro:alphasense>
+ <!-- TODO move these calibrated values into a separate file loaded by the xacro -->
+  <link name="os_imu">
+    <visual>
+      <geometry>
+        <box size="1e-3 1e-3 1e-3" />
+      </geometry>
+      <material name="black">
+        <color rgba="0 0 0 1" />
+      </material>
+    </visual>
+  </link>
+  <!-- obtained from Kalibr which is different with the datasheet-->
+  <joint name="os_imu_joint" type="fixed">
+    <origin xyz="-0.05072 -0.02064 -0.04077" rpy="3.13503 -0.00927 -0.00483"/>
+    <parent link="imu_link" />
+    <child link="os_imu" />
+  </joint>
   <link name="body">
     <visual>
